Commit message: feat(safety): 完善工业级多车协同避障与双雷达融合逻辑
1. 修复安全底层逻辑 (C++)：
   - 修复急停信号(DI11)被定位解锁信号(DI3)强行覆盖的安全漏洞。
   - 消除 DataINHandler 中 1.5s 强行恢复速度的死锁隐患。
   - 解决 sstop 变量作用域引起的编译报错。
2. 优化避障算法模块 (safety_protection)：
   - 修复 obstacle_handle 多传感器数据互相覆盖问题，引入最高优先级仲裁与 0.5s 防抖锁存。
   - 剔除 Obstacle_subfunction 中硬编码的 point_quantity，修复 speed2 初始值导致的参数漏加载。
3. 强化仿真适配 (Python & YAML)：
   - 重写 dual_lidar_fusion.py，加入 <0.1m 盲区死锁与 inf 补点，彻底解决推车走盲区问题。
   - 重写 obs_to_datain_bridge.py，加入 3 秒防抖锁存，解决雷达 0/1 抖动导致的刹车抽搐。
   - 调整 para_con.yaml 适配仿真小车尺寸与安全包络框。
4. 优化导航层：
   - URDF 前轮摩擦系数归零，完美模拟差速万向轮。
   - loop_8_shape.py 修复换任务时 pathflag 不重置导致的死机问题。

File: src/agv_sim_gazebo/urdf/agv.xacro (robot description, xacro)
@@ -79,14 +79,22 @@
   </joint>
   <!-- 激光雷达 -->
-  <link name="lidar_link">
-    <visual>
-      <geometry><cylinder radius="0.05" length="0.1"/></geometry>
-      <material name="yellow"/>
-    </visual>
+    <!-- ==================== 双雷达模型 ==================== -->
+  <!-- 左雷达 -->
+  <link name="lidar_left">
+    <visual><geometry><cylinder radius="0.05" length="0.1"/></geometry><material name="yellow"/></visual>
     <inertial><mass value="0.5"/><inertia ixx="0.01" ixy="0" ixz="0" iyy="0.01" iyz="0" izz="0.01"/></inertial>
   </link>
-  <joint name="lidar_joint" type="fixed">
-    <parent link="base_link"/><child link="lidar_link"/>
-    <origin xyz="0 0 ${base_height/2 + 0.1}" rpy="0 0 0"/>
+  <joint name="lidar_left_joint" type="fixed">
+    <parent link="base_link"/><child link="lidar_left"/>
+    <origin xyz="0.5 0 0.5" rpy="0 0 0"/>
+  </joint>
+  <!-- 右雷达 -->
+  <link name="lidar_right">
+    <visual><geometry><cylinder radius="0.05" length="0.1"/></geometry><material name="yellow"/></visual>
+    <inertial><mass value="0.5"/><inertia ixx="0.01" ixy="0" ixz="0" iyy="0.01" iyz="0" izz="0.01"/></inertial>
+  </link>
+  <joint name="lidar_right_joint" type="fixed">
+    <parent link="base_link"/><child link="lidar_right"/>
+    <origin xyz="-0.5 0 0.5" rpy="0 0 0"/>
   </joint>
   <!-- ==================== Gazebo 专属配置区 ==================== -->
@@ -124,27 +132,31 @@
   <!-- 激光雷达插件 -->
   <!-- 绝对稳妥的官方 2D 雷达插件 -->
-  <gazebo reference="lidar_link">
-    <sensor type="ray" name="lidar">
-      <pose>0 0 0 0 0 0</pose>
-      <visualize>true</visualize>
+    <!-- 左侧雷达插件，输出到 /scan_left -->
+  <gazebo reference="lidar_left">
+    <sensor type="ray" name="lidar_sensor_left">
+      <visualize>false</visualize>
       <update_rate>10</update_rate>
       <ray>
-        <scan>
-          <horizontal>
-            <samples>360</samples>
-            <resolution>1</resolution>
-            <min_angle>-3.14159</min_angle>
-            <max_angle>3.14159</max_angle>
-          </horizontal>
-        </scan>
-        <range>
-          <min>0.3</min>
-          <max>30.0</max>
-        </range>
+        <scan><horizontal><samples>360</samples><min_angle>-3.14159</min_angle><max_angle>3.14159</max_angle></horizontal></scan>
+        <range><min>0.3</min><max>30.0</max></range>
       </ray>
-      <!-- 使用最基础的激光插件，直接输出 /scan -->
-      <plugin name="gazebo_ros_laser" filename="libgazebo_ros_laser.so">
-        <topicName>/scan</topicName>
-        <frameName>lidar_link</frameName>
+      <plugin name="gazebo_ros_laser_left" filename="libgazebo_ros_laser.so">
+        <topicName>/scan_left</topicName>
+        <frameName>lidar_left</frameName>
+      </plugin>
+    </sensor>
+  </gazebo>
+  <!-- 右侧雷达插件，输出到 /scan_right -->
+  <gazebo reference="lidar_right">
+    <sensor type="ray" name="lidar_sensor_right">
+      <visualize>false</visualize>
+      <update_rate>10</update_rate>
+      <ray>
+        <scan><horizontal><samples>360</samples><min_angle>-3.14159</min_angle><max_angle>3.14159</max_angle></horizontal></scan>
+        <range><min>0.3</min><max>30.0</max></range>
+      </ray>
+      <plugin name="gazebo_ros_laser_right" filename="libgazebo_ros_laser.so">
+        <topicName>/scan_right</topicName>
+        <frameName>lidar_right</frameName>
       </plugin>
     </sensor>
